Commit message: add fixed tendon virtual roots

File: source/se3_rl_lab/se3_rl_lab/assets/robots/serialleg/urdf/serialleg_closed_chain_complex_collision.urdf (robot description, URDF)
Before this commit: robot serialleg_closed_chain_complex_collision, 11 links, 10 joints
Links:
- added link l_tendon_mount_Link, mass 0.0001
- added link r_tendon_mount_Link, mass 0.0001
- link base_link: mass 10.74541262 -> 10.74521262
- link lf0_Link: mass 0.32242010 -> 0.3224201
- link rf0_Link: mass 0.32242010 -> 0.3224201
Joints:
- added joint l_tendon_root_Joint: type revolute, parent base_link, child l_tendon_mount_Link, origin xyz=0 0 0 rpy=0 0 0, axis 0 1 0, limit lower=-0.0001 upper=0.0001 effort=40 velocity=0.1
- added joint r_tendon_root_Joint: type revolute, parent base_link, child r_tendon_mount_Link, origin xyz=0 0 0 rpy=0 0 0, axis 0 -1 0, limit lower=-0.0001 upper=0.0001 effort=40 velocity=0.1
- joint l_drive_bar_Joint: parent base_link -> l_tendon_mount_Link
- joint lf0_Joint: parent base_link -> l_tendon_mount_Link
- joint r_drive_bar_Joint: parent base_link -> r_tendon_mount_Link
- joint rf0_Joint: parent base_link -> r_tendon_mount_Link
